File: The Typeuwu PCB/keys.kicad_sch (KiCad schematic)
At the start: 268 parts, among them U1 Multi_Hotswap_with_RGB, U10 Multi_Hotswap_with_RGB, U100 Multi_Hotswap_with_RGB, U101 Multi_Hotswap_with_RGB, U102 Multi_Hotswap_with_RGB, U103 Multi_Hotswap_with_RGB, U104 Multi_Hotswap_with_RGB, U105 Multi_Hotswap_with_RGB, U11 Multi_Hotswap_with_RGB, U12 Multi_Hotswap_with_RGB, U13 Multi_Hotswap_with_RGB, U14 Multi_Hotswap_with_RGB, U15 Multi_Hotswap_with_RGB, U16 Multi_Hotswap_with_RGB, U17 Multi_Hotswap_with_RGB, U18 Multi_Hotswap_with_RGB, U19 Multi_Hotswap_with_RGB, U2 Multi_Hotswap_with_RGB, U20 Multi_Hotswap_with_RGB, U21 Multi_Hotswap_with_RGB, U22 Multi_Hotswap_with_RGB, U23 Multi_Hotswap_with_RGB, U24 Multi_Hotswap_with_RGB, U25 Multi_Hotswap_with_RGB, U26 Multi_Hotswap_with_RGB, U27 Multi_Hotswap_with_RGB, U28 Multi_Hotswap_with_RGB, U29 Multi_Hotswap_with_RGB, U3 Multi_Hotswap_with_RGB, U30 Multi_Hotswap_with_RGB, U31 Multi_Hotswap_with_RGB, U32 Multi_Hotswap_with_RGB, U33 Multi_Hotswap_with_RGB, U34 Multi_Hotswap_with_RGB, U35 Multi_Hotswap_with_RGB, U36 Multi_Hotswap_with_RGB, U37 Multi_Hotswap_with_RGB, U38 Multi_Hotswap_with_RGB, U39 Multi_Hotswap_with_RGB, U4 Multi_Hotswap_with_RGB, U40 Multi_Hotswap_with_RGB, U41 Multi_Hotswap_with_RGB, U42 Multi_Hotswap_with_RGB, U43 Multi_Hotswap_with_RGB, U44 Multi_Hotswap_with_RGB, U45 Multi_Hotswap_with_RGB, U46 Multi_Hotswap_with_RGB, U47 Multi_Hotswap_with_RGB, U48 Multi_Hotswap_with_RGB, U49 Multi_Hotswap_with_RGB, U5 Multi_Hotswap_with_RGB, U50 Multi_Hotswap_with_RGB, U51 Multi_Hotswap_with_RGB, U52 Multi_Hotswap_with_RGB, U53 Multi_Hotswap_with_RGB, U54 Multi_Hotswap_with_RGB, U55 Multi_Hotswap_with_RGB, U56 Multi_Hotswap_with_RGB, U57 Multi_Hotswap_with_RGB, U58 Multi_Hotswap_with_RGB, U59 Multi_Hotswap_with_RGB, U6 Multi_Hotswap_with_RGB, U60 Multi_Hotswap_with_RGB, U61 Multi_Hotswap_with_RGB, U62 Multi_Hotswap_with_RGB, U63 Multi_Hotswap_with_RGB, U64 Multi_Hotswap_with_RGB, U65 Multi_Hotswap_with_RGB, U66 Multi_Hotswap_with_RGB, U67 Multi_Hotswap_with_RGB, U68 Multi_Hotswap_with_RGB, U69 Multi_Hotswap_with_RGB, U7 Multi_Hotswap_with_RGB, U70 Multi_Hotswap_with_RGB, U71 Multi_Hotswap_with_RGB, U72 Multi_Hotswap_with_RGB, U8 Multi_Hotswap_with_RGB, U9 Multi_Hotswap_with_RGB, U90 Multi_Hotswap_with_RGB, U91 Multi_Hotswap_with_RGB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

Commit message: Board V1 Rev 2
Connections:
- net DIN: now reaches R14.2
Changed lines of the file:
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@@
+    (stroke (width 0) (type default))
+  )
+  (wire (pts (xy 747.395 231.14) (xy 740.41 231.14))
     (stroke (width 0) (type default))
   )
@@
     )
   )
+  (global_label "DIN" (shape input) (at 747.395 231.14 0) (fields_autoplaced)
+    (effects (font (size 1.27 1.27)) (justify left))
+    (property "Intersheetrefs" "${INTERSHEET_REFS}" (at 753.5061 231.14 0)
+      (effects (font (size 1.27 1.27)) (justify left) hide)
+    )
+  )
