File: The Typeuwu PCB/controller.kicad_sch (KiCad schematic)
At the start: 39 parts, among them J1 USB_C_Receptacle_USB2.0, J2 DEBUG, SW1 BOOT, SW2 RESET, U201 RP2040, U202 W25Q128JVS, U203 AP2112K-3.3, U73 SRV05-4, Y1 NX3225SA-12.000000MHZ

Commit message: Board V1 Rev 2
Parts:
- added C17: 100nF, Capacitor_SMD:C_0603_1608Metric, symbol Device:C
- added IC1: LSF0204QPWRQ1, SamacSys_Parts:SOP65P640X120-14N, symbol SamacSys_Parts:LSF0204QPWRQ1
- added R17, R18, R19, R20: 2k2, Resistor_SMD:R_0603_1608Metric, symbol Device:R
- added R21: 1k, Resistor_SMD:R_0603_1608Metric, symbol Device:R
- D01: footprint SamacSys:CD214AB240LR -> Diodes:CD214A-B240LR
- renumbered D02 to DL1, D03 to DL2
Connections:
- net +3V3: now also IC1.1 (VREF_A), R17.1, R18.1
- net +5V: now also C17.1, IC1.14 (VREF_B), R19.1, R20.1, R21.1; no longer C15.1, D01.1 (K)
- net GND: now also C17.2, IC1.7 (GND)
- net I2C0_SCL: now also IC1.13 (B1), R19.2; no longer U201.7 (GPIO5)
- net I2C0_SDA: now also IC1.12 (B2), R20.2; no longer U201.6 (GPIO4)
- net DIN_3V3: now reaches U201.3 (GPIO1)
- net DIN_3V3: now also IC1.4 (A3)
- net I2C1_SCL: no longer names the net of U201.5 (GPIO3)
- net I2C1_SDA: no longer names the net of U201.4 (GPIO2)
- new net: IC1.8 (EN), R21.2
- new net 5V_USB: C15.1, D01.1 (K)
- new net DIN: IC1.11 (B3)
- new net I2C0_SCL_3V3: IC1.2 (A1), R17.2, U201.7 (GPIO5)
- new net I2C0_SDA_3V3: IC1.3 (A2), R18.2, U201.6 (GPIO4)
- no-connect marks 5 -> 10

Commit message: added first module
Parts:
- D01: footprint Diodes:CD214A-B240LR -> Diode_custom:CD214A-B240LR
- IC1: footprint SamacSys_Parts:SOP65P640X120-14N -> SamacSys:SOP65P640X120-14N
- R10, R11: value R -> 1k
Connections:
- net OUT2_FLAG: now reaches U201.4 (GPIO2)
- net OUT1_FLAG: now reaches U201.5 (GPIO3)
- no-connect marks 10 -> 8
Changed lines of the file:
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@@
   (no_connect (at 180.34 105.41))
   (no_connect (at 180.34 107.95))
-  (no_connect (at 94.615 55.88))
   (no_connect (at 94.615 96.52))
   (no_connect (at 76.835 182.245))
   (no_connect (at 109.855 179.705))
   (no_connect (at 76.835 179.705))
-  (no_connect (at 94.615 58.42))
   (no_connect (at 109.855 182.245))
   (wire (pts (xy 103.505 18.415) (xy 103.505 20.32))
@@
     (stroke (width 0) (type default))
   )
+  (wire (pts (xy 94.615 55.88) (xy 96.52 55.88))
+    (stroke (width 0) (type default))
+  )
   (wire (pts (xy 191.77 83.82) (xy 193.675 83.82))
     (stroke (width 0) (type default))
@@
     (stroke (width 0) (type default))
   )
-  (wire (pts (xy 94.615 63.5) (xy 109.22 63.5))
+  (wire (pts (xy 94.615 63.5) (xy 96.52 63.5))
     (stroke (width 0) (type default))
   )
@@
     (stroke (width 0) (type default))
   )
-  (wire (pts (xy 94.615 60.96) (xy 109.22 60.96))
+  (wire (pts (xy 94.615 60.96) (xy 96.52 60.96))
     (stroke (width 0) (type default))
   )
@@
   )
   (wire (pts (xy 189.865 82.55) (xy 191.77 82.55))
+    (stroke (width 0) (type default))
+  )
+  (wire (pts (xy 96.52 58.42) (xy 94.615 58.42))
     (stroke (width 0) (type default))
   )
@@
     (effects (font (size 1.27 1.27)) (justify left bottom))
   )
-  (label "I2C0_SCL_3V3" (at 108.585 63.5 180) (fields_autoplaced)
-    (effects (font (size 1.27 1.27)) (justify right bottom))
-  )
   (label "QSPI_SD0" (at 32.385 73.66 0) (fields_autoplaced)
     (effects (font (size 1.27 1.27)) (justify left bottom))
@@
     (effects (font (size 1.27 1.27)) (justify left bottom))
   )
-  (label "I2C0_SDA_3V3" (at 108.585 60.96 180) (fields_autoplaced)
-    (effects (font (size 1.27 1.27)) (justify right bottom))
-  )
   (label "SWCLK" (at 267.335 20.955 0) (fields_autoplaced)
     (effects (font (size 1.27 1.27)) (justify left bottom))
@@
     (effects (font (size 1.27 1.27)) (justify left))
     (property "Intersheetrefs" "${INTERSHEET_REFS}" (at 107.1063 53.34 0)
+      (effects (font (size 1.27 1.27)) (justify left) hide)
+    )
+  )
+  (global_label "OUT2_FLAG" (shape bidirectional) (at 96.52 55.88 0) (fields_autoplaced)
+    (effects (font (size 1.27 1.27)) (justify left))
+    (property "Intersheetrefs" "${INTERSHEET_REFS}" (at 110.8181 55.88 0)
       (effects (font (size 1.27 1.27)) (justify left) hide)
     )
@@
     )
   )
-  (global_label "I2C0_SCL_3V3" (shape bidirectional) (at 109.22 63.5 0) (fields_autoplaced)
-    (effects (font (size 1.27 1.27)) (justify left))
-    (property "Intersheetrefs" "${INTERSHEET_REFS}" (at 126.4813 63.5 0)
-      (effects (font (size 1.27 1.27)) (justify left) hide)
-    )
-  )
-  (global_label "I2C0_SDA_3V3" (shape bidirectional) (at 109.22 60.96 0) (fields_autoplaced)
-    (effects (font (size 1.27 1.27)) (justify left))
-    (property "Intersheetrefs" "${INTERSHEET_REFS}" (at 126.5418 60.96 0)
+  (global_label "I2C0_SCL_3V3" (shape bidirectional) (at 96.52 63.5 0) (fields_autoplaced)
+    (effects (font (size 1.27 1.27)) (justify left))
+    (property "Intersheetrefs" "${INTERSHEET_REFS}" (at 113.7813 63.5 0)
+      (effects (font (size 1.27 1.27)) (justify left) hide)
+    )
+  )
+  (global_label "I2C0_SDA_3V3" (shape bidirectional) (at 96.52 60.96 0) (fields_autoplaced)
+    (effects (font (size 1.27 1.27)) (justify left))
+    (property "Intersheetrefs" "${INTERSHEET_REFS}" (at 113.8418 60.96 0)
       (effects (font (size 1.27 1.27)) (justify left) hide)
     )
@@
     )
   )
+  (global_label "OUT1_FLAG" (shape bidirectional) (at 96.52 58.42 0) (fields_autoplaced)
+    (effects (font (size 1.27 1.27)) (justify left))
+    (property "Intersheetrefs" "${INTERSHEET_REFS}" (at 110.8181 58.42 0)
+      (effects (font (size 1.27 1.27)) (justify left) hide)
+    )
+  )
   (global_label "ROW6" (shape input) (at 96.52 83.82 0) (fields_autoplaced)
     (effects (font (size 1.27 1.27)) (justify left))
@@
       (effects (font (size 1.27 1.27)) (justify left))
     )
-    (property "Value" "R" (at 230.505 40.64 0)
+    (property "Value" "1k" (at 230.505 40.64 0)
       (effects (font (size 1.27 1.27)) (justify left))
     )
@@
       (effects (font (size 1.27 1.27)) (justify left))
     )
-    (property "Value" "R" (at 243.84 40.64 0)
+    (property "Value" "1k" (at 243.84 40.64 0)
       (effects (font (size 1.27 1.27)) (justify left))
     )
@@
       (effects (font (size 1.27 1.27)))
     )
-    (property "Footprint" "Diodes:CD214A-B240LR" (at 194.945 77.47 0)
+    (property "Footprint" "Diode_custom:CD214A-B240LR" (at 194.945 77.47 0)
       (effects (font (size 1.27 1.27)) hide)
     )
@@
       (effects (font (size 1.27 1.27)))
     )
-    (property "Footprint" "SamacSys_Parts:SOP65P640X120-14N" (at 106.045 167.005 0)
-      (effects (font (size 1.27 1.27)) (justify left) hide)
-    )
+    (property "Footprint" "SamacSys:SOP65P640X120-14N" (at 106.045 167.005 0)
+      (effects (font (size 1.27 1.27)) (justify left) hide)
+    )
