File: The Typeuwu PCB/connectors.kicad_sch (KiCad schematic)
At the start: 14 parts, among them J3 Conn_01x04, J4 Conn_01x04, J5 Conn_01x04, J6 Conn_01x04

Commit message: Board V1 Rev 2
Parts:
- added D01 (x2): CD214A-B240LR, Diodes:CD214A-B240LR, symbol Device:D_Schottky
- added H1, H2, H3, H4, H5, H6, H7, H8: MountingHole, MountingHole:MountingHole_3.2mm_M3_DIN965_Pad, symbol Mechanical:MountingHole
- added J7: Battery mod, Connector_Harwin:Harwin_M20-89005xx_1x05_P2.54mm_Horizontal, symbol Connector_Generic:Conn_01x05
- added J8, J9: Conn_01x02, Connectors:POGO Magnetic 2 Pin 2,8mm Horizontal, symbol Connector_Generic:Conn_01x02
- added U74: SRV05-4, Package_TO_SOT_SMD:SOT-23-6, symbol Power_Protection:SRV05-4
Connections:
- net +5V: now also J7.5 (Pin_5)
- net GND: now also J7.1 (Pin_1), J8.1 (Pin_1), J9.1 (Pin_1)
- net I2C0_SCL: now also J7.2 (Pin_2), U74.1 (IO1)
- net I2C0_SDA: now also J7.3 (Pin_3), U74.6 (IO4)
- new net: D01.2 (A), J8.2 (Pin_2)
- new net: D01.2 (A), J9.2 (Pin_2)
- new net 5V_USB: D01.1 (K), D01.1 (K), J7.4 (Pin_4)
- no-connect marks 0 -> 2
Other:
- note added: "Bridge 5V and 5V_USB if NOT using the Battery Module. Marked as BAT BYPASS on PCB."
- moved on the sheet: J3, J4, J5, J6

Commit message: added first module
Parts:
- D01: footprint Diodes:CD214A-B240LR -> Diode_custom:CD214A-B240LR
- J3, J4, J5, J6: footprint Connector_Custom:POGO Magnetic 4 Pin Horizontal -> Connector_custom:POGO Magnetic 4 Pin 2,2mm Horizontal
- J7: value Battery mod -> M20-8900505
- J8, J9: footprint Connectors:POGO Magnetic 2 Pin 2,8mm Horizontal -> Connector_custom:POGO Magnetic 2 Pin 2,8mm Horizontal
Changed lines of the file:
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@@
       (effects (font (size 1.27 1.27)))
     )
-    (property "Footprint" "Diodes:CD214A-B240LR" (at 84.455 118.745 0)
+    (property "Footprint" "Diode_custom:CD214A-B240LR" (at 84.455 118.745 0)
       (effects (font (size 1.27 1.27)) hide)
     )
@@
       (effects (font (size 1.27 1.27)) (justify left))
     )
-    (property "Footprint" "Connectors:POGO Magnetic 2 Pin 2,8mm Horizontal" (at 94.615 140.335 0)
+    (property "Footprint" "Connector_custom:POGO Magnetic 2 Pin 2,8mm Horizontal" (at 94.615 140.335 0)
       (effects (font (size 1.27 1.27)) hide)
     )
@@
       (effects (font (size 1.27 1.27)) (justify left))
     )
-    (property "Footprint" "Connectors:POGO Magnetic 2 Pin 2,8mm Horizontal" (at 94.615 121.285 0)
+    (property "Footprint" "Connector_custom:POGO Magnetic 2 Pin 2,8mm Horizontal" (at 94.615 121.285 0)
       (effects (font (size 1.27 1.27)) hide)
     )
@@
       (effects (font (size 1.27 1.27)) (justify left))
     )
-    (property "Footprint" "Connector_Custom:POGO Magnetic 4 Pin Horizontal" (at 34.29 90.17 0)
+    (property "Footprint" "Connector_custom:POGO Magnetic 4 Pin 2,2mm Horizontal" (at 34.29 90.17 0)
       (effects (font (size 1.27 1.27)) hide)
     )
@@
       (effects (font (size 1.27 1.27)) (justify left))
     )
-    (property "Footprint" "Connector_Custom:POGO Magnetic 4 Pin Horizontal" (at 34.29 138.43 0)
+    (property "Footprint" "Connector_custom:POGO Magnetic 4 Pin 2,2mm Horizontal" (at 34.29 138.43 0)
       (effects (font (size 1.27 1.27)) hide)
     )
@@
       (effects (font (size 1.27 1.27)))
     )
-    (property "Footprint" "Diodes:CD214A-B240LR" (at 84.455 137.795 0)
+    (property "Footprint" "Diode_custom:CD214A-B240LR" (at 84.455 137.795 0)
       (effects (font (size 1.27 1.27)) hide)
     )
@@
       (effects (font (size 1.27 1.27)))
     )
-    (property "Value" "Battery mod" (at 34.29 156.845 0)
+    (property "Value" "M20-8900505" (at 34.29 156.845 0)
       (effects (font (size 1.27 1.27)))
     )
@@
       (effects (font (size 1.27 1.27)) (justify left))
     )
-    (property "Footprint" "Connector_Custom:POGO Magnetic 4 Pin Horizontal" (at 34.29 114.3 0)
+    (property "Footprint" "Connector_custom:POGO Magnetic 4 Pin 2,2mm Horizontal" (at 34.29 114.3 0)
       (effects (font (size 1.27 1.27)) hide)
     )
@@
       (effects (font (size 1.27 1.27)) (justify left))
     )
-    (property "Footprint" "Connector_Custom:POGO Magnetic 4 Pin Horizontal" (at 34.29 66.04 0)
-      (effects (font (size 1.27 1.27)) hide)
-    )
+    (property "Footprint" "Connector_custom:POGO Magnetic 4 Pin 2,2mm Horizontal" (at 34.29 66.04 0)
+      (effects (font (size 1.27 1.27)) hide)
+    )

Commit message: update to I2C and MIDI Interface
Other:
- note added: "Ups, forgot VCC and GND"
Changed lines of the file:
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@@
     (stroke (width 0) (type default))
+  )
+  (text "Ups, forgot VCC and GND" (at 69.85 77.47 0)
+    (effects (font (size 1.27 1.27)) (justify left bottom))
   )
   (text "Bridge 5V and 5V_USB if NOT using\nthe Battery Module. Marked as BAT BYPASS on PCB."
