File: Modules/Numpad/Numpad/Numpad.kicad_pcb (KiCad board)
At the start: 2 copper layers, 126 x 126 mm, 84 parts, among them J1 Display 1, J2 AVR-ISP-6, J3 Display 2, J4 Conn_01x04, J5 Conn_01x04, J6 Conn_01x04, J7 Conn_01x04, U1 Multi_Hotswap_with_RGB, U10 Multi_Hotswap_with_RGB, U11 Multi_Hotswap_with_RGB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

Commit message: firmware working version and 3D update
Parts:
- J4, J5, J6, J7: footprint Connectors:POGO Magnetic 4 Pin 2,2mm Horizontal -> Connector_custom:POGO Magnetic 4 Pin 2,2mm Horizontal
Other:
- board text added: "Green Yellow Blue"
- board text added: "Red White Black"
