File: Modules/Numpad/Numpad/controller.kicad_sch (KiCad schematic)
At the start: 28 parts, among them J1 Display 1, J2 AVR-ISP-6, J3 Display 2, J6 Conn_01x04, U18 ATmega328PB-A, Y1 ABLS-16.000MHZ-D-3-Y-T

Commit message: firmware working version and 3D update
Parts:
- J6: footprint Connectors:POGO Magnetic 4 Pin 2,2mm Horizontal -> Connector_custom:POGO Magnetic 4 Pin 2,2mm Horizontal
Changed lines of the file:
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@@
       (effects (font (size 1.27 1.27)) (justify left))
     )
-    (property "Footprint" "Connectors:POGO Magnetic 4 Pin 2,2mm Horizontal" (at 266.7 151.765 0)
+    (property "Footprint" "Connector_custom:POGO Magnetic 4 Pin 2,2mm Horizontal" (at 266.7 151.765 0)
       (effects (font (size 1.27 1.27)) hide)
     )
@@
       (effects (font (size 1.27 1.27)) (justify left))
     )
-    (property "Footprint" "Connectors:POGO Magnetic 4 Pin 2,2mm Horizontal" (at 266.7 127 0)
+    (property "Footprint" "Connector_custom:POGO Magnetic 4 Pin 2,2mm Horizontal" (at 266.7 127 0)
       (effects (font (size 1.27 1.27)) hide)
     )
@@
       (effects (font (size 1.27 1.27)) (justify left))
     )
-    (property "Footprint" "Connectors:POGO Magnetic 4 Pin 2,2mm Horizontal" (at 267.335 76.835 0)
+    (property "Footprint" "Connector_custom:POGO Magnetic 4 Pin 2,2mm Horizontal" (at 267.335 76.835 0)
       (effects (font (size 1.27 1.27)) hide)
     )
@@
       (effects (font (size 1.27 1.27)) (justify left))
     )
-    (property "Footprint" "Connectors:POGO Magnetic 4 Pin 2,2mm Horizontal" (at 267.335 101.6 0)
-      (effects (font (size 1.27 1.27)) hide)
-    )
+    (property "Footprint" "Connector_custom:POGO Magnetic 4 Pin 2,2mm Horizontal" (at 267.335 101.6 0)
+      (effects (font (size 1.27 1.27)) hide)
+    )
